File: schematics/prototipo/arduino_datalogger.kicad_sch (KiCad schematic)
At the start: 9 parts, among them SW1 SW_Push, U1 DHT22

Commit message: Eliminado PCB y footprints personalizadas
Decidimos hacer el prototipo en perfboard, así que ya no es necesario lo anterior
Parts:
- removed A2: SD card module, Custom_Modules:MicroSD_Module, symbol Custom_Modules:MicroSD_Module
- removed A3: RTC module, Custom_Modules:RTCDS3231, symbol Custom_Modules:RTCDS3231
- added A2: RTC Module, symbol Custom_Modules:RTCDS3231
- added A3: MicroSD Module, symbol Custom_Modules:MicroSD_Module
- A1: value Arduino_Nano_v3.x -> Arduino Nano ATmega 328P
- SW1: value SW_Push -> Push Button
Connections:
- net +5V: now also A2.5 (VCC), A3.5 (VCC)
- net CS: now also A3.1 (CS)
- net GND: now also A2.6 (GND), A3.6 (GND)
- net MISO: now also A3.4 (MISO)
- net MOSI: now also A3.3 (MOSI)
- net SCK: now also A3.2 (SCK)
- net SCL: now also A2.3 (SCL)
- net SDA: now also A2.4 (SDA)
- net SQW: now also A2.2 (SQW)

Commit message: Corregidas conexiones de LCD
VO estaba conectado a Vcc con una R de 220 (debe ir a GND con R de 1K).
Vss tenia una R de 1K (debe tener una de 220).
Parts:
- R1: value 1K -> 220
- R2: value 220 -> 1k
Connections:
- net +5V: no longer R2.1
- net GND: now also R2.1
Other:
- moved on the sheet: A1, DS1, R1, R2, R3, SW1, U1
