File: board/arduino_datalogger.kicad_sch (KiCad schematic)
At the start: 9 parts, among them SW1 Push Button, U1 DHT22

Commit message: Traslation of schematic to English
Other:
- company: Lab. Biología de los Artrópodos - FaCENA - UNNE -> (none)
- title: Prototipo datalogger con Arduino -> Arduino based datalogger prototipe
Changed lines of the file:
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@@
   (paper "A5")
   (title_block
-    (title "Prototipo datalogger con Arduino")
-    (date "2023-12-02")
+    (title "Arduino based datalogger prototipe")
+    (date "2023-12-18")
     (rev "0.1")
-    (company "Lab. Biología de los Artrópodos - FaCENA - UNNE")
-    (comment 1 "Autor/es: Lucas J. Mina, Dario D. Larrea y Miryam P. Damborsky")
+    (comment 1 "Author/s: Lucas J. Mina, Dario D. Larrea y Miryam P. Damborsky")
   )
   (junction (at 121.92 58.42) (diameter 0) (color 0 0 0 0)
